Commit message: Fix wheels placement

File: src/robobox/urdf/robobox.xacro (robot description, xacro)
@@ -5,7 +5,7 @@
     <xacro:property name="height" value="0.778" />
     <xacro:property name="pi" value="3.1415" />
-    <xacro:property name="small_wheel_radius" value="0.05" />
-    <xacro:property name="small_wheel_length" value="0.02" />
-    <xacro:property name="big_wheel_radius" value="0.15" />
+    <xacro:property name="small_wheel_radius" value="0.07" />
+    <xacro:property name="small_wheel_length" value="0.04" />
+    <xacro:property name="big_wheel_radius" value="0.14" />
     <xacro:property name="big_wheel_length" value="0.1" />
     <xacro:property name="camera_size" value="0.05" />
@@ -68,5 +68,5 @@
             </geometry>
         </collision>
-        <xacro:default_inertial mass="10" />
+        <xacro:default_inertial mass="100" />
         <gazebo reference="base_link">
             <material>Gazebo/Red</material>
@@ -93,9 +93,9 @@
         <child link="base_link" />
     </joint>
-    <xacro:wheel prefix="front" suffix="left" offset_x="30.3" offset_y="0.1" offset_z="${small_wheel_radius}" radius="${small_wheel_radius}" length="${small_wheel_length}"/>
-    <xacro:wheel prefix="front" suffix="right" offset_x="30.3" offset_y="-0.1" offset_z="${small_wheel_radius}" radius="${small_wheel_radius}" length="${small_wheel_length}"/>
-    <xacro:wheel prefix="back" suffix="left" offset_x="-1" offset_y="0.5" offset_z="-${big_wheel_radius / 2}" radius="${big_wheel_radius}" length="${big_wheel_length}"/>
-    <xacro:wheel prefix="back" suffix="right" offset_x="-1" offset_y="-0.5" offset_z="-${big_wheel_radius / 2}" radius="${big_wheel_radius}" length="${big_wheel_length}"/>
-  <!-- Camera -->
+    <xacro:wheel prefix="front" suffix="mid" offset_x="15.5" offset_y="0" offset_z="0" radius="${small_wheel_radius}" length="${small_wheel_length}"/>
+    <xacro:wheel prefix="back" suffix="mid" offset_x="-15.5" offset_y="0" offset_z="0" radius="${small_wheel_radius}" length="${small_wheel_length}"/>
+    <xacro:wheel prefix="mid" suffix="left" offset_x="0" offset_y="0.5" offset_z="-${big_wheel_radius / 2}" radius="${big_wheel_radius}" length="${big_wheel_length}"/>
+    <xacro:wheel prefix="mid" suffix="right" offset_x="0" offset_y="-0.5" offset_z="-${big_wheel_radius / 2}" radius="${big_wheel_radius}" length="${big_wheel_length}"/>
+  <!-- Camera >
   <joint name="camera_joint" type="fixed">
     <axis xyz="0 1 0" />
@@ -159,8 +159,5 @@
       </plugin>
     </sensor>
-  </gazebo>
-  <!-- Noise is sampled independently per pixel on each frame.
-               That pixel's noise value is added to each of its color
-               channels, which at that point lie in the range [0,1]. -->
+  </gazebo-->
    <!-- Hokuyo Laser -->
     <joint name="hokuyo_joint" type="fixed">
@@ -227,122 +224,4 @@
     </sensor>
   </gazebo>
-    <!--link name="hokuyo_link">
-      <pose>0.05 0 0.11 0 0 0</pose>
-      <inertial>
-        <inertia>
-          <ixx>1e-6</ixx>
-          <ixy>0</ixy>
-          <ixz>0</ixz>
-          <iyy>1e-6</iyy>
-          <iyz>0</iyz>
-          <izz>1e-6</izz>
-        </inertia>
-        <mass>1e-5</mass>
-      </inertial>
-      <collision name="collision">
-        <pose>0 0 0.5 0 0 0</pose>
-        <geometry>
-          <box>
-            <size>0.1 0.1 0.1</size>
-          </box>
-        </geometry>
-      </collision>
-      <visual name="visual">
-        <geometry>
-          <mesh>
-            <uri>model://hokuyo/meshes/hokuyo.dae</uri>
-          </mesh>
-        </geometry>
-      </visual>
-      <sensor name="laser" type="ray">
-        <pose>0.01 0 0.0175 0 -0 0</pose>
-        <ray>
-          <scan>
-            <horizontal>
-              <samples>640</samples>
-              <resolution>1</resolution>
-              <min_angle>-2.26889</min_angle>
-              <max_angle>2.268899</max_angle>
-            </horizontal>
-          </scan>
-          <range>
-            <min>0.08</min>
-            <max>10</max>
-            <resolution>0.01</resolution>
-          </range>
-        </ray>
-        <plugin name="laser" filename="libRayPlugin.so" />
-        <always_on>1</always_on>
-        <update_rate>30</update_rate>
-        <visualize>true</visualize>
-      </sensor>
-    </link>
-     <joint name="hokuyo_joint" type="revolute">
-        <parent link="base_link"/>
-        <child link="hokuyo_link"/>
-        <axis xyz="0 1 0" />
-        <limit effort="1000.0" lower="0.0" upper="0.0" velocity="0.5"/>
-      <axis>
-        <xyz>0 1 0</xyz>
-        <limit>
-          <upper>0</upper>
-          <lower>0</lower>
-        </limit>
-      </axis>
-    </joint-->
-    <!--link name="laser_scan_link" type="laser">
- <inertial>
-      <mass value="0.5" />
-      <origin xyz="0 0 0" />
-      <inertia ixx="0.3"  ixy="0.3"  ixz="0.3" iyy="0.3"  iyz="0.3"  izz="0.3" />
-     </inertial>
-     <visual>
-       <origin xyz="0 0 0" rpy="0 0 0"/>
-       <geometry>
-         <cylinder length="0.1" radius="0.05" />
-       </geometry>
-     </visual>
-     <collision>
-      <origin xyz="0 0 0" rpy="0 0 0"/>
-       <geometry>
-         <cylinder length="0.1" radius="0.05" />
-       </geometry>
-     </collision>
-  </link>
-<joint name="laser_to_base_link" type="fixed">
-  <origin xyz="0.25 0 0.32" rpy="0 0 0" />
-  <parent link="base_link" />
-  <child link="laser_scan_link"/>
-</joint>
-   <gazebo reference="laser_scan_link">
-  <sensor:ray name="laser_scan_link">
-     <rayCount>683</rayCount>
-     <rangeCount>683</rangeCount>
-     <laserCount>1</laserCount>
-         <origin>0.0 0.0 0.0</origin>
-         <displayRays>true</displayRays>
-         <minAngle>-105</minAngle>
-         <maxAngle>105</maxAngle>
-         <minRange>0.06</minRange>
-         <maxRange>4.0</maxRange>
-         <resRange>0.01</resRange>
-         <updateRate>10.0</updateRate>
-         <controller:gazebo_ros_laser name="gazebo_ros_base_scan_link_controller" plugin="libgazebo_ros_laser.so">
-                <gaussianNoise>0.005</gaussianNoise>
-                <alwaysOn>true</alwaysOn>
-                <updateRate>20.0</updateRate>
-                <topicName>base_scan/scan</topicName>
-                <frameName>laser_scan_link</frameName>
-                <interface:laser name="gazebo_ros_base_scan_link_iface"/>
-         </controller:gazebo_ros_laser>
-        </sensor:ray>
-    </gazebo>
-  <gazebo>
-   <controller:gazebo_ros_controller_manager name="gazebo_ros_controller_manager" plugin="libgazebo_ros_controller_manager.so">
-      <alwaysOn>true</alwaysOn>
-      <updateRate>1000.0</updateRate>
-      <interface:audio name="gazebo_ros_controller_manager_dummy_iface" />
-    </controller:gazebo_ros_controller_manager>
-  </gazebo-->
     <gazebo>
       <plugin name="gazebo_ros_control" filename="libgazebo_ros_control.so" />
@@ -350,10 +229,10 @@
         <alwaysOn>true</alwaysOn>
         <updateRate>100.0</updateRate>
-        <leftJoint>back_left_wheel_joint</leftJoint>
-        <rightJoint>back_right_wheel_joint</rightJoint>
+        <leftJoint>mid_left_wheel_joint</leftJoint>
+        <rightJoint>mid_right_wheel_joint</rightJoint>
         <wheelSeparation>${width}</wheelSeparation>
-        <wheelDiameter>${2.5 * big_wheel_radius}</wheelDiameter>
+        <wheelDiameter>${2 * big_wheel_radius}</wheelDiameter>
         <wheelTorque>100</wheelTorque>
-        <wheelAcceleration>0</wheelAcceleration>
+        <wheelAcceleration>10</wheelAcceleration>
         <commandTopic>cmd_vel</commandTopic>
         <odometryTopic>odom</odometryTopic>
@@ -362,39 +241,3 @@
       </plugin>
     </gazebo>
-   <!--gazebo>
-    <plugin name="gazebo_ros_control" filename="libgazebo_ros_control.so" />
-    <plugin name="skid_steer_drive_controller" filename="libgazebo_ros_skid_steer_drive.so">
-      <alwaysOn>1</alwaysOn>
-      <updateRate>100.0</updateRate>
-      <leftFrontJoint>front_left_wheel_joint</leftFrontJoint>
-      <rightFrontJoint>front_right_wheel_joint</rightFrontJoint>
-      <leftRearJoint>back_left_wheel_joint</leftRearJoint>
-      <rightRearJoint>back_right_wheel_joint</rightRearJoint>
-      <wheelSeparation>${width}</wheelSeparation>
-      <wheelDiameter>${2.5 * big_wheel_radius}</wheelDiameter>
-      <torque>100</torque>
-      <broadcastTF>1</broadcastTF>
-      <commandTopic>cmd_vel</commandTopic>
-      <odometryFrame>odom</odometryFrame>
-      <odometryTopic>odom</odometryTopic>
-      <robotBaseFrame>base_footprint</robotBaseFrame>
-    </plugin>
-  </gazebo-->
-    <!--gazebo>
-        <plugin name="skid_steer_drive_controller" filename="libgazebo_ros_skid_steer_drive.so">
-            <alwaysOn>true</alwaysOn>
-            <updateRate>100.0</updateRate>
-            <robotNamespace>/</robotNamespace>
-            <leftJoint>back_left_wheel_joint</leftJoint>
-            <rightJoint>back_right_wheel_joint</rightJoint>
-            <wheelSeparation>0.4</wheelSeparation>
-            <wheelDiameter>0.2</wheelDiameter>
-            <robotBaseFrame>base_link</robotBaseFrame>
-            <torque>1</torque>
-            <odometryTopic>odom</odometryTopic>
-            <odometryFrame>odom</odometryFrame>
-            <topicName>cmd_vel</topicName>
-            <broadcastTF>0</broadcastTF>
-        </plugin>
-    </gazebo-->
 </robot>

Commit message: Update code base

File: src/robobox/urdf/robobox.xacro (robot description, xacro)
@@ -16,44 +16,37 @@
         <inertial>
             <mass value="${mass}" />
+            <origin xyz=" 0 0 0"/>
             <inertia ixx="1.0" ixy="0.0" ixz="0.0" iyy="1.0" iyz="0.0" izz="1.0" />
         </inertial>
     </xacro:macro>
-    <xacro:macro name="wheel" params="prefix suffix offset_x offset_y offset_z radius length">
+    <xacro:macro name="wheel" params="prefix suffix ratio_x ratio_y offset_z wheel_radius wheel_length joint_type">
         <link name="${prefix}_${suffix}_wheel">
             <visual>
-                <origin xyz="0 0 0" rpy="${pi/2} 0 0" />
+                <origin xyz="0 0 0" rpy="0 ${pi/2} ${pi/2}" />
                 <geometry>
-                    <cylinder radius="${radius}" length="${length}" />
+                    <cylinder radius="${wheel_radius}" length="${wheel_length}" />
                 </geometry>
                 <material name="black" />
-                <origin xyz=" 0 0 0" rpy="0 0 0" />
             </visual>
             <collision>
-                <origin xyz="0 0 0" rpy="${pi/2} 0 0" />
+                <origin xyz="0 0 0" rpy="0 ${pi/2} ${pi/2}" />
                 <geometry>
-                    <cylinder radius="${radius}" length="${length}" />
+                    <cylinder radius="${wheel_radius}" length="${wheel_length}" />
                 </geometry>
-                <material name="black" />
-                <origin xyz=" 0 0 0" rpy="0 0 0" />
             </collision>
-            <xacro:default_inertial mass="1" />
-            <gazebo reference="${prefix}_${suffix}_wheel">
-                <material>Gazebo/Black</material>
-            </gazebo>
+            <xacro:default_inertial mass="0.01" />
         </link>
-        <joint name="${prefix}_${suffix}_wheel_joint" type="continuous">
-            <axis xyz="0 1 0" rpy="0 0 0" />
+        <joint name="${prefix}_${suffix}_wheel_joint" type="${joint_type}">
+            <axis xyz="0 1 0" />
             <parent link="base_link" />
             <child link="${prefix}_${suffix}_wheel" />
-            <origin xyz="${length * offset_x} ${width * offset_y} -${height/2 + offset_z}" rpy="0 0 0" />
+            <origin xyz="${length * ratio_x} ${width * ratio_y} -${height/2 + offset_z}" rpy="0 0 0" />
         </joint>
-        <!--transmission name="${prefix}_${suffix}_trans">
-              <type>transmission_interface/SimpleTransmission</type>
-              <joint name="${prefix}_${suffix}_wheel_hinge"/>
-              <actuator name="${prefix}_${suffix}_Motor">
-                    <hardwareInterface>EffortJointInterface</hardwareInterface>
-                    <mechanicalReduction>10</mechanicalReduction>
-              </actuator>
-        </transmission-->
+    </xacro:macro>
+    <xacro:macro name="small_wheel" params="prefix suffix ratio_x">
+        <xacro:wheel prefix="${prefix}" suffix="${suffix}" ratio_x="${ratio_x}" ratio_y="0" offset_z="-${small_wheel_radius}" wheel_radius="${small_wheel_radius}" wheel_length="${small_wheel_length}" joint_type="fixed"/>
+    </xacro:macro>
+    <xacro:macro name="big_wheel" params="prefix suffix ratio_y">
+        <xacro:wheel prefix="${prefix}" suffix="${suffix}" ratio_x="0" ratio_y="${ratio_y}" offset_z="-${big_wheel_radius / 2}" wheel_radius="${big_wheel_radius}" wheel_length="${big_wheel_length}" joint_type="continuous"/>
     </xacro:macro>
     <link name="base_link">
@@ -93,9 +86,9 @@
         <child link="base_link" />
     </joint>
-    <xacro:wheel prefix="front" suffix="mid" offset_x="15.5" offset_y="0" offset_z="0" radius="${small_wheel_radius}" length="${small_wheel_length}"/>
-    <xacro:wheel prefix="back" suffix="mid" offset_x="-15.5" offset_y="0" offset_z="0" radius="${small_wheel_radius}" length="${small_wheel_length}"/>
-    <xacro:wheel prefix="mid" suffix="left" offset_x="0" offset_y="0.5" offset_z="-${big_wheel_radius / 2}" radius="${big_wheel_radius}" length="${big_wheel_length}"/>
-    <xacro:wheel prefix="mid" suffix="right" offset_x="0" offset_y="-0.5" offset_z="-${big_wheel_radius / 2}" radius="${big_wheel_radius}" length="${big_wheel_length}"/>
-  <!-- Camera >
+    <xacro:small_wheel prefix="front" suffix="mid" ratio_x="0.5" />
+    <xacro:small_wheel prefix="back" suffix="mid" ratio_x="-0.5" />
+    <xacro:big_wheel prefix="mid" suffix="left" ratio_y="0.5" />
+    <xacro:big_wheel prefix="mid" suffix="right" ratio_y="-0.5" />
+  <!-- Camera -->
   <joint name="camera_joint" type="fixed">
     <axis xyz="0 1 0" />
@@ -159,13 +152,12 @@
       </plugin>
     </sensor>
-  </gazebo-->
-   <!-- Hokuyo Laser -->
+  </gazebo>
+   <!-- Hokuyo Laser >
     <joint name="hokuyo_joint" type="fixed">
         <axis xyz="0 1 0" />
-        <origin xyz="${length/2} 0 ${height/2}" rpy="0 0 0"/>
+        <origin xyz="${length/2} 0 ${height/2+0.1}" rpy="0 0 0"/>
         <parent link="base_link"/>
         <child link="hokuyo_link"/>
       </joint>
-  <!-- Hokuyo Laser -->
   <link name="hokuyo_link">
     <collision>
@@ -188,5 +180,4 @@
     </inertial>
   </link>
-  <!-- hokuyo -->
   <gazebo reference="hokuyo_link">
     <sensor type="gpu_ray" name="head_hokuyo_sensor">
@@ -199,19 +190,15 @@
             <samples>720</samples>
             <resolution>1</resolution>
-            <min_angle>-1.570796</min_angle>
-            <max_angle>1.570796</max_angle>
+            <min_angle>-3.1570796</min_angle>
+            <max_angle>3.1570796</max_angle>
           </horizontal>
         </scan>
         <range>
           <min>0.10</min>
-          <max>30.0</max>
+          <max>300.0</max>
           <resolution>0.01</resolution>
         </range>
         <noise>
           <type>gaussian</type>
-          <!-- Noise parameters based on published spec for Hokuyo laser
-               achieving "+-30mm" accuracy at range < 10m.  A mean of 0.0m and
-               stddev of 0.01m will put 99.7% of samples within 0.03m of the true
-               reading. -->
           <mean>0.0</mean>
           <stddev>0.01</stddev>
@@ -223,6 +210,66 @@
       </plugin>
     </sensor>
-  </gazebo>
-    <gazebo>
+  </gazebo-->
+<!-- Hokuyo LIDAR for simulation -->
+  <xacro:macro name="hokuyo_laser">
+    <gazebo reference="base_laser_link">
+      <sensor type="ray" name="laser">
+        <pose>0 0 0 0 0 0</pose>
+        <visualize>true</visualize>
+        <update_rate>40</update_rate>
+        <ray>
+          <scan>
+            <horizontal>
+              <samples>720</samples>
+              <resolution>1</resolution>
+              <min_angle>-3.1415</min_angle>
+              <max_angle>3.1415</max_angle>
+            </horizontal>
+          </scan>
+          <range>
+            <min>0.10</min>
+            <max>30.0</max>
+            <resolution>0.01</resolution>
+          </range>
+          <noise>
+            <type>Gaussian</type>
+            <mean>0.0</mean>
+            <stddev>0.01</stddev>
+          </noise>
+        </ray>
+        <plugin name="hokuyo_node" filename="libgazebo_ros_laser.so">
+          <topicName>/robobox/laser/scan</topicName>
+          <frameName>base_laser_link</frameName>
+        </plugin>
+      </sensor>
+    </gazebo>
+  </xacro:macro>
+  <xacro:macro name="sensor_hokuyo">
+    <joint name="laser" type="fixed">
+      <origin xyz="${length/2} 0 ${height/2+0.1}" rpy="0 0 0"/>
+      <!--origin xyz="0.15 0.0 0.360" rpy="3.14159 0.0 0.0" /-->
+      <parent link="base_link" />
+      <child link="base_laser_link" />
+    </joint>
+    <link name="base_laser_link">
+      <visual>
+        <geometry>
+          <box size="0.00 0.05 0.06" />
+        </geometry>
+        <material name="black" />
+      </visual>
+      <inertial>
+        <mass value="0.000001" />
+        <origin xyz="0 0 0" />
+        <inertia ixx="0.0001" ixy="0.0" ixz="0.0"
+          iyy="0.0001" iyz="0.0"
+          izz="0.0001" />
+      </inertial>
+    </link>
+    <!-- Set up laser gazebo details -->
+    <hokuyo_laser />
+  </xacro:macro>
+    <sensor_hokuyo />
+    <!--gazebo>
       <plugin name="gazebo_ros_control" filename="libgazebo_ros_control.so" />
       <plugin name="differential_drive_controller" filename="libgazebo_ros_diff_drive.so">
@@ -240,4 +287,4 @@
         <robotBaseFrame>base_footprint</robotBaseFrame>
       </plugin>
-    </gazebo>
+    </gazebo-->
 </robot>
